File: HDK/Commander/Commander.kicad_sch (KiCad schematic)
At the start: 36 parts, among them J1 SWD, SW1 BOOT0, SW2 NRST, U1 STM32G431CBU6, Y1 32.768K, Y1 8M

Commit message: Update Commander
Connections:
- net VBAT+: now also D1.3; no longer D1.2
- net VBAT_Pin: now also D1.2; no longer D1.3
Changed lines of the file:
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@@
 (kicad_sch (version 20230121) (generator eeschema)
   (paper "A4")
-  (title_block
-    (rev "1.1v")
-  )
   (junction (at 141.605 19.685) (diameter 0) (color 0 0 0 0)
   )
@@
     (effects (font (size 1.5 1.5) italic) (justify left bottom))
   )
-  (label "VBAT_Pin" (at 262.89 123.19 0) (fields_autoplaced)
-    (effects (font (size 1.27 1.27)) (justify left bottom))
-  )
   (label "LCD.CS" (at 264.16 45.72 180) (fields_autoplaced)
     (effects (font (size 1.27 1.27) italic) (justify right bottom))
@@
     (effects (font (size 1.27 1.27) italic) (justify left bottom))
   )
+  (label "VBAT_Pin" (at 247.65 132.08 0) (fields_autoplaced)
+    (effects (font (size 1.27 1.27)) (justify left bottom))
+  )
+  (label "VBAT+" (at 262.89 123.19 0) (fields_autoplaced)
+    (effects (font (size 1.27 1.27)) (justify left bottom))
+  )
   (label "NRST" (at 120.015 70.485 180) (fields_autoplaced)
     (effects (font (size 1.27 1.27) italic) (justify right bottom))
@@
     (effects (font (size 1.27 1.27) italic) (justify left bottom))
   )
-  (label "VBAT+" (at 247.65 132.08 0) (fields_autoplaced)
-    (effects (font (size 1.27 1.27)) (justify left bottom))
-  )
   (label "PB4" (at 30.48 93.345 0) (fields_autoplaced)
